Commit message: end-effector WIP
the end effector is able to be controlled independently of the usual
move group, but the motion is not quite correct. Looks like there should
be some modifications to the joint positions in
robotiq_arg2f_140_model_macro.xacro

File: urdf/robotiq_arg2f_140_model_macro.xacro (robot description, xacro)
@@ -18,5 +18,5 @@
         <origin xyz="0 0 0" rpy="0 0 0" />
         <geometry>
-          <mesh filename="package://robotiq_2f_140_gripper_visualization/meshes/visual/robotiq_arg2f_${stroke}_outer_knuckle.stl" />
+          <mesh filename="package://ece383-final-project/meshes/visual/robotiq_arg2f_${stroke}_outer_knuckle.stl" />
         </geometry>
         <material name="">
@@ -27,5 +27,5 @@
         <origin xyz="0 0 0" rpy="0 0 0" />
         <geometry>
-          <mesh filename="package://robotiq_2f_140_gripper_visualization/meshes/collision/robotiq_arg2f_${stroke}_outer_knuckle.stl" />
+          <mesh filename="package://ece383-final-project/meshes/collision/robotiq_arg2f_${stroke}_outer_knuckle.stl" />
         </geometry>
       </collision>
@@ -48,5 +48,5 @@
         <origin xyz="0 0 0" rpy="0 0 0" />
         <geometry>
-          <mesh filename="package://robotiq_2f_140_gripper_visualization/meshes/visual/robotiq_arg2f_${stroke}_outer_finger.stl" />
+          <mesh filename="package://ece383-final-project/meshes/visual/robotiq_arg2f_${stroke}_outer_finger.stl" />
         </geometry>
         <material name="">
@@ -57,5 +57,5 @@
         <origin xyz="0 0 0" rpy="0 0 0" />
         <geometry>
-          <mesh filename="package://robotiq_2f_140_gripper_visualization/meshes/collision/robotiq_arg2f_${stroke}_outer_finger.stl" />
+          <mesh filename="package://ece383-final-project/meshes/collision/robotiq_arg2f_${stroke}_outer_finger.stl" />
         </geometry>
       </collision>
@@ -78,5 +78,5 @@
         <origin xyz="0 0 0" rpy="0 0 0" />
         <geometry>
-          <mesh filename="package://robotiq_2f_140_gripper_visualization/meshes/visual/robotiq_arg2f_${stroke}_inner_knuckle.stl" />
+          <mesh filename="package://ece383-final-project/meshes/visual/robotiq_arg2f_${stroke}_inner_knuckle.stl" />
         </geometry>
         <material name="">
@@ -87,5 +87,5 @@
         <origin xyz="0 0 0" rpy="0 0 0" />
         <geometry>
-          <mesh filename="package://robotiq_2f_140_gripper_visualization/meshes/collision/robotiq_arg2f_${stroke}_inner_knuckle.stl" />
+          <mesh filename="package://ece383-final-project/meshes/collision/robotiq_arg2f_${stroke}_inner_knuckle.stl" />
         </geometry>
       </collision>
@@ -108,5 +108,5 @@
         <origin xyz="0 0 0" rpy="0 0 0" />
         <geometry>
-          <mesh filename="package://robotiq_2f_140_gripper_visualization/meshes/visual/robotiq_arg2f_${stroke}_inner_finger.stl" />
+          <mesh filename="package://ece383-final-project/meshes/visual/robotiq_arg2f_${stroke}_inner_finger.stl" />
         </geometry>
         <material name="">
@@ -117,5 +117,5 @@
         <origin xyz="0 0 0" rpy="0 0 0" />
         <geometry>
-          <mesh filename="package://robotiq_2f_140_gripper_visualization/meshes/collision/robotiq_arg2f_${stroke}_inner_finger.stl" />
+          <mesh filename="package://ece383-final-project/meshes/collision/robotiq_arg2f_${stroke}_inner_finger.stl" />
         </geometry>
       </collision>
@@ -181,5 +181,5 @@
     </joint>
   </xacro:macro>
-  <xacro:include filename="$(find robotiq_2f_140_gripper_visualization)/urdf/robotiq_arg2f.xacro" />
+  <xacro:include filename="$(find ece383-final-project)/urdf/robotiq_arg2f.xacro" />
   <xacro:macro name="finger_joint" params="prefix">
     <joint name="${prefix}finger_joint" type="revolute">
@@ -188,5 +188,5 @@
       <child link="${prefix}left_outer_knuckle" />
       <axis xyz="-1 0 0" />
-      <limit lower="0" upper="0.7" velocity="2.0" effort="1000" />
+      <limit lower="-5" upper="5" velocity="2.0" effort="1000" />
     </joint>
     <xacro:finger_joints prefix="${prefix}" fingerprefix="left" reflect="1.0"/>
@@ -198,5 +198,5 @@
       <child link="${prefix}right_outer_knuckle" />
       <axis xyz="1 0 0" />
-      <limit lower="0" upper="0.725" velocity="2.0" effort="1000" />
+      <limit lower="-5" upper="5" velocity="2.0" effort="1000" />
     <mimic joint="${prefix}finger_joint" multiplier="-1" offset="0" />
     </joint>
@@ -212,4 +212,11 @@
     <gazebo>
         <!-- loading plugin: mimic joints works in gazebo now-->
+        <plugin filename="libroboticsgroup_gazebo_mimic_joint_plugin.so" name="${prefix}mimic_robotiq_85_1">
+          <joint>${prefix}finger_joint</joint>
+          <mimicJoint>${prefix}left_outer_knuckle_joint</mimicJoint>
+          <multiplier>1.0</multiplier>
+          <!--<multiplier>-1.0</multiplier>-->
+          <!--<offset>0.0</offset>-->
+        </plugin>
         <plugin filename="libroboticsgroup_gazebo_mimic_joint_plugin.so" name="${prefix}mimic_robotiq_85_4">
           <joint>${prefix}finger_joint</joint>

Commit message: WIP but EE fingers correct

File: urdf/robotiq_arg2f_140_model_macro.xacro (robot description, xacro)
@@ -211,44 +211,36 @@
     <xacro:robotiq_arg2f_transmission prefix="${prefix}"/>
     <gazebo>
-        <!-- loading plugin: mimic joints works in gazebo now-->
-        <plugin filename="libroboticsgroup_gazebo_mimic_joint_plugin.so" name="${prefix}mimic_robotiq_85_1">
-          <joint>${prefix}finger_joint</joint>
-          <mimicJoint>${prefix}left_outer_knuckle_joint</mimicJoint>
+        <plugin filename="libroboticsgroup_gazebo_mimic_joint_plugin.so" name="${prefix}mimic_robotiq_85_4">
+          <joint>${prefix}finger_joint</joint>
+          <mimicJoint>${prefix}right_outer_knuckle_joint</mimicJoint>
+          <multiplier>-1.0</multiplier>
+          <!--<multiplier>-1.0</multiplier>-->
+          <!--<offset>0.0</offset>-->
+        </plugin>
+        <plugin filename="libroboticsgroup_gazebo_mimic_joint_plugin.so" name="${prefix}mimic_robotiq_85_2">
+          <joint>${prefix}finger_joint</joint>
+          <mimicJoint>${prefix}left_inner_finger_joint</mimicJoint>
           <multiplier>1.0</multiplier>
+          <!--<multiplier>1.0</multiplier>-->
+          <!--<offset>0.0</offset>-->
+        </plugin>
+        <plugin filename="libroboticsgroup_gazebo_mimic_joint_plugin.so" name="${prefix}mimic_robotiq_85_6">
+          <joint>${prefix}finger_joint</joint>
+          <mimicJoint>${prefix}right_inner_finger_joint</mimicJoint>
+          <multiplier>1.0</multiplier>
+          <!--<multiplier>1.0</multiplier>-->
+          <!--<offset>0.0</offset>-->
+        </plugin>
+          <plugin filename="libroboticsgroup_gazebo_mimic_joint_plugin.so" name="${prefix}mimic_robotiq_85_3">
+          <joint>${prefix}finger_joint</joint>
+          <mimicJoint>${prefix}left_inner_knuckle_joint</mimicJoint>
+          <multiplier>-1.0</multiplier>
           <!--<multiplier>-1.0</multiplier>-->
           <!--<offset>0.0</offset>-->
         </plugin>
-        <plugin filename="libroboticsgroup_gazebo_mimic_joint_plugin.so" name="${prefix}mimic_robotiq_85_4">
-          <joint>${prefix}finger_joint</joint>
-          <mimicJoint>${prefix}right_outer_knuckle_joint</mimicJoint>
-          <multiplier>1.0</multiplier>
-          <!--<multiplier>-1.0</multiplier>-->
-          <!--<offset>0.0</offset>-->
-        </plugin>
-        <plugin filename="libroboticsgroup_gazebo_mimic_joint_plugin.so" name="${prefix}mimic_robotiq_85_2">
-          <joint>${prefix}finger_joint</joint>
-          <mimicJoint>${prefix}left_inner_finger_joint</mimicJoint>
+        <plugin filename="libroboticsgroup_gazebo_mimic_joint_plugin.so" name="${prefix}mimic_robotiq_85_5">
+          <joint>${prefix}finger_joint</joint>
+          <mimicJoint>${prefix}right_inner_knuckle_joint</mimicJoint>
           <multiplier>-1.0</multiplier>
-          <!--<multiplier>1.0</multiplier>-->
-          <!--<offset>0.0</offset>-->
-        </plugin>
-        <plugin filename="libroboticsgroup_gazebo_mimic_joint_plugin.so" name="${prefix}mimic_robotiq_85_6">
-          <joint>${prefix}finger_joint</joint>
-          <mimicJoint>${prefix}right_inner_finger_joint</mimicJoint>
-          <multiplier>-1.0</multiplier>
-          <!--<multiplier>1.0</multiplier>-->
-          <!--<offset>0.0</offset>-->
-        </plugin>
-          <plugin filename="libroboticsgroup_gazebo_mimic_joint_plugin.so" name="${prefix}mimic_robotiq_85_3">
-          <joint>${prefix}finger_joint</joint>
-          <mimicJoint>${prefix}left_inner_knuckle_joint</mimicJoint>
-          <multiplier>1.0</multiplier>
-          <!--<multiplier>-1.0</multiplier>-->
-          <!--<offset>0.0</offset>-->
-        </plugin>
-        <plugin filename="libroboticsgroup_gazebo_mimic_joint_plugin.so" name="${prefix}mimic_robotiq_85_5">
-          <joint>${prefix}finger_joint</joint>
-          <mimicJoint>${prefix}right_inner_knuckle_joint</mimicJoint>
-          <multiplier>1.0</multiplier>
           <!--<multiplier>-1.0</multiplier>-->
           <!--<offset>0.0</offset>-->

File: urdf/robotiq_arg2f_transmission.xacro (robot description, xacro)
@@ -6,4 +6,5 @@
       <joint name="${prefix}finger_joint">
         <hardwareInterface>hardware_interface/PositionJointInterface</hardwareInterface>
+        <!-- <hardwareInterface>hardware_interface/EffortJointInterface</hardwareInterface> -->
       </joint>
       <actuator name="${prefix}finger_joint_motor">
