Commit message: add notes to function, move camera

File: urdf/my_camera.xacro (robot description, xacro)
@@ -7,5 +7,5 @@
             <axis xyz="1 0 0" />
             <!-- <origin xyz="${camera_link} 0 ${height3 - axel_offset*2}" rpy="0 0 0"/> -->
-            <origin xyz="0.5 -1 0" rpy="0 0 1.57"/>
+            <origin xyz="0.3 -1 0.17" rpy="0 0 1.57"/>
             <parent link="world"/>
             <child link="camera_link"/>
@@ -37,5 +37,6 @@
             <update_rate>30.0</update_rate>
             <camera name="head">
-                <horizontal_fov>1.3962634</horizontal_fov>
+                <!-- <horizontal_fov>1.3962634</horizontal_fov> -->
+                <horizontal_fov>0.45</horizontal_fov>
                 <image>
                 <width>800</width>

Commit message: optimize token placement (cartesian + better math) also disable some annoying log messages

File: urdf/my_camera.xacro (robot description, xacro)
@@ -24,5 +24,4 @@
             <box size="${camera_link} ${camera_link} ${camera_link}"/>
             </geometry>
-            <material name="red"/>
             </visual>
             <inertial>
