Commit message: add token (designed by Reyna) and modify inertia
token was added in red and yellow versions, and the inertia of the board
was modified such that it would allow the token to fall in

File: urdf/board.xacro (robot description, xacro)
@@ -29,11 +29,11 @@
             </collision>
             <inertial>
-                <mass value="1e-5" />
+                <mass value="1e-1" />
                 <origin xyz="0 0 0" rpy="0 0 0"/>
-                <inertia ixx="1e-6" ixy="0" ixz="0" iyy="1e-6" iyz="0" izz="1e-6" />
+                <inertia ixx="1e-1" ixy="0" ixz="0" iyy="1e-1" iyz="0" izz="1e-1" />
             </inertial>
         </link>
         <gazebo reference="board_link">
-            <material>Gazebo/Yellow</material>
+            <material>Gazebo/Blue</material>
         </gazebo>
     </xacro:macro>

Commit message: pick up token and place in board WIP
move board closer to robot, make disc holder and token heavier,
add GraspFix plugin, and simplify token geometry

File: urdf/board.xacro (robot description, xacro)
@@ -6,5 +6,5 @@
             <axis xyz="1 0 0" />
             <!-- <origin xyz="${camera_link} 0 ${height3 - axel_offset*2}" rpy="0 0 0"/> -->
-            <origin xyz="0.5 -0.5 0" rpy="0 0 0"/>
+            <origin xyz="0.25 -0.25 0" rpy="0 0 0"/>
             <parent link="world"/>
             <child link="board_link"/>

File: urdf/disc_holder.urdf (robot description, URDF)
Before this commit: robot None, 1 links, 0 joints
Links:
- link single_disc_holder_link: mass 1 -> 10

File: urdf/token_red.urdf (robot description, URDF)
Before this commit: robot None, 1 links, 0 joints
Links:
- link token_link: mass 1e-2 -> 1

File: urdf/token_yellow.urdf (robot description, URDF)
Before this commit: robot None, 1 links, 0 joints
Links:
- link token_link: mass 1e-2 -> 1

File: urdf/ur.xacro (robot description, xacro)
@@ -105,3 +105,20 @@
   <xacro:include filename="$(find ece383-final-project)/urdf/modifications.xacro"/>
   <xacro:ece383/>
+  <gazebo>
+    <plugin name="gazebo_grasp_fix" filename="libgazebo_grasp_fix.so">
+        <arm>
+          <arm_name>random_name</arm_name>
+          <palm_link> wrist_3_link  </palm_link>
+          <gripper_link> left_inner_finger </gripper_link>
+          <gripper_link> right_inner_finger </gripper_link>
+        </arm>
+      <forces_angle_tolerance>100</forces_angle_tolerance>
+      <update_rate>10</update_rate>
+      <grip_count_threshold>2</grip_count_threshold>
+      <max_grip_count>20</max_grip_count>
+      <release_tolerance>0.005</release_tolerance>
+      <disable_collisions_on_attach>true</disable_collisions_on_attach>
+      <contact_topic>__default_topic__</contact_topic>
+    </plugin>
+  </gazebo>
 </robot>

Commit message: improve token manipulation, physics

File: urdf/board.xacro (robot description, xacro)
@@ -29,7 +29,7 @@
             </collision>
             <inertial>
-                <mass value="1e-1" />
+                <mass value="10" />
                 <origin xyz="0 0 0" rpy="0 0 0"/>
-                <inertia ixx="1e-1" ixy="0" ixz="0" iyy="1e-1" iyz="0" izz="1e-1" />
+                <inertia ixx="1" ixy="0" ixz="0" iyy="1" iyz="0" izz="1" />
             </inertial>
         </link>

Commit message: general geometry cleanup, ros launch fix
 - decrease board mass because a higher mass makes the tokens fall thru
sometimes (idk why)
 - make token position centered on the token
 - wait to start ROS until previous session has ended
 - add help file so `from help import *` in python is easy
 - add forward kinematics to get end effector pos

File: urdf/board.xacro (robot description, xacro)
@@ -29,7 +29,7 @@
             </collision>
             <inertial>
-                <mass value="10" />
+                <mass value="1e-1" />
                 <origin xyz="0 0 0" rpy="0 0 0"/>
-                <inertia ixx="1" ixy="0" ixz="0" iyy="1" iyz="0" izz="1" />
+                <inertia ixx="1e-1" ixy="0" ixz="0" iyy="1e-1" iyz="0" izz="1e-1" />
             </inertial>
         </link>

Commit message: place tokens in all 7 columns

File: urdf/board.xacro (robot description, xacro)
@@ -6,5 +6,5 @@
             <axis xyz="1 0 0" />
             <!-- <origin xyz="${camera_link} 0 ${height3 - axel_offset*2}" rpy="0 0 0"/> -->
-            <origin xyz="0.25 -0.25 0" rpy="0 0 0"/>
+            <origin xyz="0.058 -0.25 0" rpy="0 0 0"/>
             <parent link="world"/>
             <child link="board_link"/>
@@ -13,5 +13,5 @@
         <link name="board_link">
             <visual>
-                <origin xyz="0 0 0" rpy="1.57 0 0" />
+                <origin xyz="0.112 0 0" rpy="1.57 0 0" />
                 <geometry>
                     <mesh filename="package://ece383-final-project/meshes/visual/board.stl" scale="0.001 0.001 0.001">
@@ -23,5 +23,5 @@
             </visual>
             <collision>
-                <origin xyz="0 0 0" rpy="1.57 0 0" />
+                <origin xyz="0.112 0 0" rpy="1.57 0 0" />
                 <geometry>
                     <mesh filename="package://ece383-final-project/meshes/visual/board.stl" scale="0.001 0.001 0.001"/>

Commit message: gameplay working (no CV though)

File: urdf/board.xacro (robot description, xacro)
@@ -29,5 +29,5 @@
             </collision>
             <inertial>
-                <mass value="1e-1" />
+                <mass value="1000" />
                 <origin xyz="0 0 0" rpy="0 0 0"/>
                 <inertia ixx="1e-1" ixy="0" ixz="0" iyy="1e-1" iyz="0" izz="1e-1" />
